File: sensor/sensor.kicad_pcb (KiCad board)
At the start: 2 copper layers, 1 part

Commit message: Managed to 3d print a pcb with copper tape
(also forgot to push the firmware before this)
Parts:
- added D1: LED, LED_THT:LED_D5.0mm, F.Cu at (98.6, 67.6)
- added R1: R, Resistor_THT:R_Axial_DIN0207_L6.3mm_D2.5mm_P10.16mm_Horizontal, F.Cu at (93.1, 67.6)
- added U2: ~, sensor:SHT31_breakout, F.Cu at (90.5, 78.7)
- moved U1 8.90 mm to (115.0, 75.2)
Routing:
- net +3V3: track 0.00 -> 43.7 mm
- net Net-(U1-GPIO8/SDA/LED): track 0.00 -> 11.9 mm
- net Net-(U1-GPIO9/SCL/BOOT): track 0.00 -> 11.9 mm
- net Net-(D1-A): track 0.00 -> 5.69 mm
- net Net-(D1-K): track 0.00 -> 5.52 mm
- added copper zone on F.Cu, net GND
Other:
- board outline added: 46 x 27 mm
