File: sensor/sensor.kicad_sch (KiCad schematic)
At the start: 4 parts

Commit message: Managed to 3d print a pcb with copper tape
(also forgot to push the firmware before this)
Parts:
- D1: footprint (none) -> LED_THT:LED_D5.0mm
- R1: footprint (none) -> Resistor_THT:R_Axial_DIN0207_L6.3mm_D2.5mm_P10.16mm_Horizontal
- U2: footprint (none) -> sensor:SHT31_breakout
Changed lines of the file:
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@@
 			)
 		)
-		(property "Footprint" ""
+		(property "Footprint" "Resistor_THT:R_Axial_DIN0207_L6.3mm_D2.5mm_P10.16mm_Horizontal"
 			(at 176.022 97.79 90)
 			(effects
@@
 			)
 		)
-		(property "Footprint" ""
+		(property "Footprint" "sensor:SHT31_breakout"
 			(at 186.69 68.58 0)
 			(effects
@@
 			)
 		)
-		(property "Footprint" ""
+		(property "Footprint" "LED_THT:LED_D5.0mm"
 			(at 189.23 92.71 0)
 			(effects
